File: robo_pendulo.kicad_sch (KiCad schematic)
At the start: 51 parts, among them J1 Conn_01x02, J10 Conn_01x04, J11 Conn_01x04, J2 Conn_01x09, J4 Conn_01x02_Male, J5 Conn_01x02_Male, J6 Conn_01x02_Male, J7 Conn_01x02_Male, J8 Conn_02x13_Odd_Even, SW1 SW_SPST, U1 LM324, U2 L298HN, U3 LM324, U4 HC-05, U5 MPU-6050

Commit message: começo do desenvolvimento do leiaute
Parts:
- C2: renamed from C1; value C -> 1u
- C3: renamed from C2; value C -> 1u
- C4: renamed from C3; footprint Capacitor_SMD:C_0805_2012Metric -> Capacitor_Tantalum_SMD:CP_EIA-3216-12_Kemet-S
- C5: footprint Capacitor_SMD:C_0805_2012Metric -> Capacitor_Tantalum_SMD:CP_EIA-3216-12_Kemet-S
- D10: renamed from D8; footprint Diode_THT:D_DO-41_SOD81_P10.16mm_Horizontal -> Diode_SMD:D_SMA
- D2: renamed from D12; footprint Diode_SMD:D_SMB -> Package_TO_SOT_SMD:SOT-23
- D3: renamed from D1; footprint Diode_THT:D_DO-41_SOD81_P10.16mm_Horizontal -> Diode_SMD:D_SMA
- D4: renamed from D2; footprint Diode_THT:D_DO-41_SOD81_P10.16mm_Horizontal -> Diode_SMD:D_SMA
- D5: renamed from D3; footprint Diode_THT:D_DO-41_SOD81_P10.16mm_Horizontal -> Diode_SMD:D_SMA
- D6: renamed from D4; footprint Diode_THT:D_DO-41_SOD81_P10.16mm_Horizontal -> Diode_SMD:D_SMA
- D7: renamed from D5; footprint Diode_THT:D_DO-41_SOD81_P10.16mm_Horizontal -> Diode_SMD:D_SMA
- D8: renamed from D6; footprint Diode_THT:D_DO-41_SOD81_P10.16mm_Horizontal -> Diode_SMD:D_SMA
- D9: renamed from D7; footprint Diode_THT:D_DO-41_SOD81_P10.16mm_Horizontal -> Diode_SMD:D_SMA
- R1, R2, R3, R4: footprint Resistor_SMD:R_0805_2012Metric -> Resistor_SMD:R_1206_3216Metric
- R10: renamed from R23; value R -> 10k; footprint Resistor_SMD:R_0805_2012Metric -> Resistor_SMD:R_1206_3216Metric
- R11: renamed from R18; value R -> 47k; footprint Resistor_SMD:R_0805_2012Metric -> Resistor_SMD:R_1206_3216Metric
- R12: renamed from R17; value R -> 10k; footprint Resistor_SMD:R_0805_2012Metric -> Resistor_SMD:R_1206_3216Metric
- R13: renamed from R5; value R -> 150; footprint Resistor_SMD:R_0805_2012Metric -> Resistor_SMD:R_1206_3216Metric
- R14: renamed from R6; value R -> 150; footprint Resistor_SMD:R_0805_2012Metric -> Resistor_SMD:R_1206_3216Metric
- R15: renamed from R35; footprint Resistor_SMD:R_0805_2012Metric -> Resistor_SMD:R_1206_3216Metric
- R16: renamed from R7; footprint Resistor_SMD:R_0805_2012Metric -> Resistor_THT:R_Axial_DIN0414_L11.9mm_D4.5mm_P5.08mm_Vertical
- R17: renamed from R8; footprint Resistor_SMD:R_0805_2012Metric -> Resistor_THT:R_Axial_DIN0414_L11.9mm_D4.5mm_P5.08mm_Vertical
- R5: renamed from R20; value R -> 3k; footprint Resistor_SMD:R_0805_2012Metric -> Resistor_SMD:R_1206_3216Metric
- R6: renamed from R22; value R -> 3k; footprint Resistor_SMD:R_0805_2012Metric -> Resistor_SMD:R_1206_3216Metric
- R7: renamed from R19; value R -> 1k; footprint Resistor_SMD:R_0805_2012Metric -> Resistor_SMD:R_1206_3216Metric
- R8: renamed from R21; value R -> 1k; footprint Resistor_SMD:R_0805_2012Metric -> Resistor_SMD:R_1206_3216Metric
- R9: renamed from R24; value R -> 47k; footprint Resistor_SMD:R_0805_2012Metric -> Resistor_SMD:R_1206_3216Metric
- SW1: footprint (none) -> TerminalBlock:TerminalBlock_bornier-2_P5.08mm
- renumbered C4 to C1, D11 to D1, J6 to J3, J7 to J5, J5 to J6, J10 to J7, J11 to J8, J8 to J9, U3 to U1, U4 to U2, U2 to U3, U5 to U4
Connections:
- net +BATT: now also J1.1 (Pin_1), SW1.2 (B); no longer SW1.1 (A)
- net CURR_LM: now also R8.2; no longer R6.2
- net CURR_RM: now also R6.2; no longer R8.2
- new net BATT_IN: SW1.1 (A)
Other:
- note added: "Decoupling ceramic capacitor must be near source pins"
- moved on the sheet: J1

Commit message: Adjust board layout
Parts:
- removed J3, J4, J5, J6: Conn_01x02_Male, Connector_PinSocket_2.54mm:PinSocket_1x02_P2.54mm_Vertical, symbol Connector:Conn_01x02_Male
- added J6, J7: Conn_01x02, Connector_PinHeader_2.54mm:PinHeader_1x02_P2.54mm_Vertical, symbol Connector_Generic:Conn_01x02
- added U2: mini-DC-DC, dc-dc-converter:mini-DC-DC, symbol arduino_shields:mini-DC-DC
- C4, C5: footprint Capacitor_Tantalum_SMD:CP_EIA-3216-12_Kemet-S -> Capacitor_SMD:CP_Elec_8x10
- J1: footprint Connector_PinSocket_2.54mm:PinSocket_1x02_P2.54mm_Vertical -> Connector_AMASS:AMASS_XT60-M_1x02_P7.20mm_Vertical
- R10, R12: value 10k -> 82k
- R11, R9: value 47k -> 82k
- R16, R17: footprint Resistor_THT:R_Axial_DIN0414_L11.9mm_D4.5mm_P5.08mm_Vertical -> Resistor_THT:R_Axial_DIN0516_L15.5mm_D5.0mm_P7.62mm_Vertical
- R5, R6: value 3k -> 3k3
- R7, R8: value 1k -> 3k3
- SW1: footprint TerminalBlock:TerminalBlock_bornier-2_P5.08mm -> (none)
- renumbered J7 to J3, J8 to J4, J9 to J5, U2 to U4, U4 to U5
Connections:
- net +5V: now also D2.3 (A), U2.1 (OUT+), U2.2 (OUT+); no longer D2.2 (A), J2.2 (Pin_2)
- net +BATT: now also SW1.1 (A), U2.5 (IN+), U2.6 (IN+); no longer J1.1 (Pin_1), SW1.2 (B)
- net BATT_IN: now also J1.1 (Pin_1), SW1.2 (B); no longer SW1.1 (A)
- net CLP: now also J2.9 (Pin_9), J5.21 (Pin_21); no longer J2.1 (Pin_1)
- net CURR_LM: now also R16.2, R6.2, U3.1 (SENSE_A); no longer R17.2, R8.2, U3.15 (SENSE_B)
- net CURR_RM: now also R17.2, R8.2, U3.15 (SENSE_B); no longer R16.2, R6.2, U3.1 (SENSE_A)
- net ENC0_A: now also J5.3 (Pin_3)
- net ENC0_B: now also J5.5 (Pin_5)
- net ENC1_A: now also J5.25 (Pin_25)
- net ENC1_B: now also J5.23 (Pin_23)
- net GND: now also J2.1 (Pin_1), U2.3 (OUT-), U2.4 (OUT-), U2.7 (IN-), U2.8 (IN-); no longer J2.9 (Pin_9)
- net IMU_INT: now also J5.10 (Pin_10)
- net IMU_SCL: now also J5.6 (Pin_6)
- net IMU_SDA: now also J5.8 (Pin_8)
- net MEAS_BATT: now also J5.2 (Pin_2), U1.8; no longer U1.14
- net MEAS_LM: now also J5.4 (Pin_4)
- net MEAS_RM: now also J5.1 (Pin_1)
- net MOT_ENA: now also J5.12 (Pin_12), J5.22 (Pin_22)
- net MOT_IN1: now also J5.16 (Pin_16)
- net MOT_IN2: now also J5.14 (Pin_14)
- net MOT_IN4: now also J5.18 (Pin_18)
- net MOT_OUT1: now also J6.1 (Pin_1)
- net MOT_OUT2: now also J6.2 (Pin_2)
- net MOT_OUT3: now also J7.1 (Pin_1)
- net MOT_OUT4: now also J7.2 (Pin_2)
- net NEAR: now also J2.2 (Pin_2), J5.7 (Pin_7); no longer J2.8 (Pin_8)
- net RXB: now also J5.24 (Pin_24)
- net SS1: now also J2.7 (Pin_7), J5.17 (Pin_17); no longer J2.3 (Pin_3)
- net SS2: now also J2.6 (Pin_6), J5.15 (Pin_15); no longer J2.4 (Pin_4)
- net SS3: now also J5.13 (Pin_13)
- net SS4: now also J2.4 (Pin_4), J5.11 (Pin_11); no longer J2.6 (Pin_6)
- net SS5: now also J2.3 (Pin_3), J5.9 (Pin_9); no longer J2.7 (Pin_7)
- net TXB: now also J5.26 (Pin_26)
- net at R12.1, R14.2: now also U1.14; no longer U1.8
- net at R12.2, R7.1: now also U1.13 (-); no longer U1.9 (-)
- net at R10.1, R8.1: now also U1.12 (+); no longer U1.10 (+)
- net 5V_OUT: now reaches J5.19 (Pin_19)
- net 5V_OUT: now also D2.2 (K), J2.8 (Pin_8)
- net MOT_INB: now reaches J5.20 (Pin_20)
- net at R2.1, R3.1: now also U1.10 (+); no longer U1.12 (+)
- net at R1.1, R4.2: now also U1.9 (-); no longer U1.13 (-)
Other:
- moved on the sheet: C4, C5, D10, D2, D3, D4, D5, D6, D7, D8, D9, J1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
